File: schematic_PWRcutoff.kicad_pcb (KiCad board)
At the start: 2 copper layers, 100 x 100 mm, 44 parts, among them J1 Conn_01x02, J10 Conn_01x02, J11 Conn_01x02, J12 Conn_01x08, J13 Conn_01x08, J14 Conn_01x02, J15 Conn_01x02, J2 Conn_01x02, J3 Conn_01x02, J4 Conn_01x04, J5 Conn_01x02, J6 Conn_01x04, J7 Conn_01x02, J8 Conn_01x02, J9 Conn_01x02, K1 RAYEX-L90AS, K2 RAYEX-L90AS, Q1 Q_NMOS_GSD, Q2 Q_NMOS_GSD

Commit message: precompreate design
Parts:
- removed the D2 at (122.3, 70.2)
- removed the J1 at (91.1, 56.0)
- removed the J2 at (118.2, 46.6)
- removed J3: Conn_01x02, RDC_general:XT90-M
- removed J5: Conn_01x02, Connector_PinHeader_2.54mm:PinHeader_1x02_P2.54mm_Vertical
- removed the J8 at (91.4, 131.3)
- removed the J9 at (91.5, 137.3)
- removed REF**: KiCad-Logo2_5mm_SilkScreen, Symbol:KiCad-Logo2_5mm_SilkScreen
- added C10: 0.1uF, Capacitor_SMD:C_0603_1608Metric_Pad1.08x0.95mm_HandSolder, F.Cu at (87.2, 104.2)
- added C11: 0.1uF, Capacitor_SMD:C_0603_1608Metric_Pad1.08x0.95mm_HandSolder, F.Cu at (123.8, 52.5)
- added C12: 0.1uF, Capacitor_SMD:C_0603_1608Metric_Pad1.08x0.95mm_HandSolder, F.Cu at (83.4, 96.1)
- added C13: 0.1uF, Capacitor_SMD:C_0603_1608Metric_Pad1.08x0.95mm_HandSolder, F.Cu at (94.0, 114.0)
- added C14: 0.1uF, Capacitor_SMD:C_0603_1608Metric_Pad1.08x0.95mm_HandSolder, F.Cu at (110.1, 87.1)
- added C15: 0.1uF, Capacitor_SMD:C_0603_1608Metric_Pad1.08x0.95mm_HandSolder, F.Cu at (86.9, 89.4)
- added C16: 10uF, Capacitor_SMD:C_0603_1608Metric_Pad1.08x0.95mm_HandSolder, F.Cu at (101.9, 109.4)
- added C17: 0.1uF, Capacitor_SMD:C_0603_1608Metric_Pad1.08x0.95mm_HandSolder, F.Cu at (100.8, 108.3)
- added C18: 0.1uF, Capacitor_SMD:C_0603_1608Metric_Pad1.08x0.95mm_HandSolder, F.Cu at (114.1, 94.2)
- added C19: 10uF, Capacitor_SMD:C_0603_1608Metric_Pad1.08x0.95mm_HandSolder, F.Cu at (117.2, 95.8)
- added C2: 0.1uF, Capacitor_SMD:C_0603_1608Metric_Pad1.08x0.95mm_HandSolder, F.Cu at (141.3, 60.6)
- added C20: 22uF, Capacitor_SMD:C_0603_1608Metric_Pad1.08x0.95mm_HandSolder, F.Cu at (119.1, 106.5)
- added C21: 1000uF, Capacitor_THT:CP_Radial_D10.0mm_P5.00mm, F.Cu at (99.4, 88.1)
- added C4: 0.1uF, Capacitor_SMD:C_0603_1608Metric_Pad1.08x0.95mm_HandSolder, F.Cu at (87.5, 123.5)
- added C5: 10pF, Capacitor_SMD:C_0603_1608Metric_Pad1.08x0.95mm_HandSolder, F.Cu at (100.9, 112.8)
- added C6: 10pF, Capacitor_SMD:C_0603_1608Metric_Pad1.08x0.95mm_HandSolder, F.Cu at (96.6, 117.1)
- added C7: 10uF, Capacitor_SMD:C_0603_1608Metric_Pad1.08x0.95mm_HandSolder, F.Cu at (105.8, 108.8)
- added C8: 0.1uF, Capacitor_SMD:C_0603_1608Metric_Pad1.08x0.95mm_HandSolder, F.Cu at (91.5, 112.9)
- added C9: 0.1uF, Capacitor_SMD:C_0603_1608Metric_Pad1.08x0.95mm_HandSolder, F.Cu at (96.7, 99.7)
- added D7: LED, LED_SMD:LED_0603_1608Metric_Pad1.05x0.95mm_HandSolder, F.Cu at (122.0, 134.9)
- added D8: MA10EB045, Diode_SMD:Vishay_SMPA, F.Cu at (110.0, 93.3)
- added J14: STlink_v3, RDC_general:JTAG_box_connector, F.Cu at (82.1, 116.8)
- added JP1: Jumper, Connector_PinHeader_2.54mm:PinHeader_1x02_P2.54mm_Vertical, F.Cu at (84.0, 85.5)
- added JP2: Jumper, Connector_PinHeader_2.54mm:PinHeader_1x02_P2.54mm_Vertical, F.Cu at (94.5, 131.2)
- added JP3: Jumper, Connector_PinHeader_2.54mm:PinHeader_1x02_P2.54mm_Vertical, F.Cu at (103.4, 131.2)
- added L1: 22uH, RDC_general:CDRH6D38, F.Cu at (109.0, 99.0)
- added Q1: Q_PMOS_GSD, Package_TO_SOT_SMD:TO-252-2, F.Cu at (149.6, 56.0)
- added Q4: Q_NMOS_GSD, Package_TO_SOT_SMD:SOT-23, F.Cu at (92.9, 123.3)
- added Q5: Q_PMOS_GSD, Package_TO_SOT_SMD:SOT-23, F.Cu at (93.0, 127.0)
- added Q6: Q_NMOS_GSD, Package_TO_SOT_SMD:SOT-23, F.Cu at (102.9, 123.3)
- added Q7: Q_PMOS_GSD, Package_TO_SOT_SMD:TO-252-2, F.Cu at (118.6, 54.9)
- added Q8: Q_PMOS_GSD, Package_TO_SOT_SMD:TO-252-2, F.Cu at (149.6, 63.0)
- added Q9: Q_PMOS_GSD, Package_TO_SOT_SMD:TO-252-2, F.Cu at (111.6, 54.9)
- added R12: 10k, Resistor_SMD:R_0603_1608Metric_Pad0.98x0.95mm_HandSolder, F.Cu at (88.5, 113.2)
- added R13: 100, Resistor_SMD:R_0603_1608Metric_Pad0.98x0.95mm_HandSolder, F.Cu at (97.2, 123.3)
- added R14: 10k, Resistor_SMD:R_0603_1608Metric_Pad0.98x0.95mm_HandSolder, F.Cu at (95.7, 123.3)
- added R15: 10k, Resistor_SMD:R_0603_1608Metric_Pad0.98x0.95mm_HandSolder, F.Cu at (97.2, 127.0)
- added R16: 100, Resistor_SMD:R_0603_1608Metric_Pad0.98x0.95mm_HandSolder, F.Cu at (107.1, 123.3)
- added R17: 10k, Resistor_SMD:R_0603_1608Metric_Pad0.98x0.95mm_HandSolder, F.Cu at (105.6, 123.3)
- added R18: 10k, Resistor_SMD:R_0603_1608Metric_Pad0.98x0.95mm_HandSolder, F.Cu at (102.9, 120.8)
- added R19: 10k, Resistor_SMD:R_0603_1608Metric_Pad0.98x0.95mm_HandSolder, F.Cu at (123.8, 54.0)
- added R20: 10k, Resistor_SMD:R_0603_1608Metric_Pad0.98x0.95mm_HandSolder, F.Cu at (123.8, 55.5)
- added R21: 120, Resistor_SMD:R_0603_1608Metric_Pad0.98x0.95mm_HandSolder, F.Cu at (83.1, 82.9)
- added R22: 10k, Resistor_SMD:R_0603_1608Metric_Pad0.98x0.95mm_HandSolder, F.Cu at (95.7, 127.0)
- added R23: 10k, Resistor_SMD:R_0603_1608Metric_Pad0.98x0.95mm_HandSolder, F.Cu at (118.7, 134.9)
- added R24: 10k, Resistor_SMD:R_0603_1608Metric_Pad0.98x0.95mm_HandSolder, F.Cu at (115.4, 89.8)
- added R25: 10k, Resistor_SMD:R_0603_1608Metric_Pad0.98x0.95mm_HandSolder, F.Cu at (113.9, 89.8)
- added R26: 10k, Resistor_SMD:R_0603_1608Metric_Pad0.98x0.95mm_HandSolder, F.Cu at (100.5, 95.0)
- added R27: 10k, Resistor_SMD:R_0603_1608Metric_Pad0.98x0.95mm_HandSolder, F.Cu at (112.3, 46.0)
- added R28: 10k, Resistor_SMD:R_0603_1608Metric_Pad0.98x0.95mm_HandSolder, F.Cu at (110.9, 118.9)
- added R29: 10k, Resistor_SMD:R_0603_1608Metric_Pad0.98x0.95mm_HandSolder, F.Cu at (112.4, 118.9)
- added R30: 10k, Resistor_SMD:R_0603_1608Metric_Pad0.98x0.95mm_HandSolder, F.Cu at (113.9, 118.9)
- added R31: 10k, Resistor_SMD:R_0603_1608Metric_Pad0.98x0.95mm_HandSolder, F.Cu at (115.4, 118.9)
- added R4: 10k, Resistor_SMD:R_0603_1608Metric_Pad0.98x0.95mm_HandSolder, F.Cu at (141.3, 63.6)
- added SW1: SW_SPST, RDC_general:Toggle_switch, F.Cu at (133.1, 80.3)
- added SW2: SW_DIP_x04, Button_Switch_SMD:SW_DIP_SPSTx04_Slide_Copal_CHS-04B_W7.62mm_P1.27mm, F.Cu at (113.2, 112.3)
- added SW3: SW_SPST, RDC_general:Toggle_switch, F.Cu at (127.7, 80.3)
- added SW4: SW_SPST, Button_Switch_THT:SW_PUSH_6mm_H7.3mm, F.Cu at (80.7, 129.9)
- added U1: MCP2562-H-SN, Package_SO:SOIC-8_3.9x4.9mm_P1.27mm, F.Cu at (83.4, 91.4)
- added U2: STM32F103CBTx, Package_QFP:LQFP-48_7x7mm_P0.5mm, F.Cu at (94.0, 106.3)
- added U3: ~, Package_TO_SOT_SMD:SOT-23-6_Handsoldering, F.Cu at (110.7, 89.8)
- added U4: AZ1117-3.3, Package_TO_SOT_SMD:SOT-223-3_TabPin2, F.Cu at (118.6, 101.2)
- added U5: ~, RDC_general:MPD7K020S, F.Cu at (103.0, 71.5)
- added Y1: 12MHz, Crystal:Crystal_SMD_SeikoEpson_FA238V-4Pin_3.2x2.5mm, F.Cu at (98.8, 115.0)
- C1: value 100uF -> 1000uF; footprint Capacitor_THT:CP_Radial_D8.0mm_P5.00mm -> Capacitor_THT:CP_Radial_D16.0mm_P7.50mm
- C3: renamed from C2; footprint Capacitor_THT:CP_Radial_D18.0mm_P7.50mm -> Capacitor_THT:CP_Radial_D16.0mm_P7.50mm
- J12, J13: value Conn_01x08 -> Conn_01x02; footprint Connector_PinHeader_2.54mm:PinHeader_1x08_P2.54mm_Vertical -> Connector_JST:JST_XA_B02B-XASK-1_1x02_P2.50mm_Vertical
- J7: footprint Connector_PinHeader_2.54mm:PinHeader_1x02_P2.54mm_Vertical -> RDC_general:XT90-M
- RV1: footprint Varistor:RV_Disc_D12mm_W4.5mm_P7.5mm -> Varistor:RV_Disc_D9mm_W4.5mm_P5mm
- moved J7 98.2 mm to (142.4, 40.8)
- moved J12 53.4 mm to (92.0, 137.2), turned to 0 degrees
- moved R3 23.8 mm to (141.3, 62.1)
- moved J13 22.2 mm to (100.8, 137.2), turned to 0 degrees
- moved R5 21.8 mm to (156.3, 63.9)
- moved R2 20.4 mm to (124.3, 63.5), turned to 0 degrees
- moved RV1 19.1 mm to (128.3, 45.2), turned to 180 degrees
- moved D2 16.8 mm to (127.7, 63.5), turned to 180 degrees
- moved C1 14.1 mm to (100.9, 49.9), turned to 180 degrees
- moved J1 13.5 mm to (83.2, 52.7), turned to -90 degrees
- moved R6 10.6 mm to (125.5, 87.8)
- moved R7 10.5 mm to (125.5, 89.3)
- moved R9 10.5 mm to (125.5, 116.6)
- moved R10 10.4 mm to (125.5, 118.1)
- moved Q2 10.3 mm to (125.5, 92.1)
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- renumbered D3 to D2, D5 to D3, D7 to D5, H3 to H2, H2 to H3, J4 to J1, J15 to J10, J6 to J2, J14 to J8, J10 to J9, Q1 to Q2, Q2 to Q3, R2 to R1, R8 to R11, R4 to R2, R1 to R5, R5 to R8
Connections:
- C1 pad 1: +12V -> Logic_line_Power
- C3 pad 1: +24V -> Actuator_Power
- C3 pad 2: GNDPWR -> GND
- D2 pad 1: GNDPWR -> GND
- D4 pad 1: 12VIN -> +12V
- D6 pad 1: 12VIN -> +12V
- H2 pad 1: GNDPWR -> GND
- H4 pad 1: GNDPWR -> GND
- J1 pad 2: 12VIN -> +12V
- J1 pad 3: CANH -> Net-(J1-Pin_3)
- J1 pad 4: CANL -> Net-(J1-Pin_4)
- J10 pad 1: GNDPWR -> GND
- J11 pad 1: GNDPWR -> GND
- J12 pad 1: GND -> Net-(J12-Pin_1)
- J12 pad 2: 12VIN -> Net-(J12-Pin_2)
- J13 pad 1: GND -> Net-(J12-Pin_2)
- J13 pad 2: GND -> /EMS/Relay_Signal_OUT
- J2 pad 2: 12VIN -> +12V
- J2 pad 3: CANH -> Net-(J1-Pin_3)
- J2 pad 4: CANL -> Net-(J1-Pin_4)
- J7 pad 1: GNDPWR -> GND
- J8 pad 1: GNDPWR -> GND
- J9 pad 1: GNDPWR -> GND
- K1 pad 13: +24V -> Actuator_Power
- K1 pad A2: 12VIN -> +12V
- K2 pad 13: +24V -> Actuator_Power
- K2 pad A2: 12VIN -> +12V
- R1 pad 1: +12V -> Logic_line_Power
- R11 pad 1: 12VIN -> +12V
- R2 pad 1: +24V -> Actuator_Power
- R3 pad 1: 12VIN -> +24V
- R5 pad 1: +24V -> Actuator_Power
- R5 pad 2: GNDPWR -> GND
- R6 pad 2: /PWR_Cutoff_Relay Sheet/Relay_Coil_Signal -> /EMS/Relay_Signal_OUT
- R8 pad 1: 12VIN -> +12V
- R9 pad 2: /PWR_Cutoff_Relay Sheet/Relay_Coil_Signal -> /EMS/Relay_Signal_OUT
- RV1 pad 1: +12V -> +24V
Routing:
- net 12VIN: track 164.8 -> 0.00 mm
- net +3.3V: track 0.00 -> 136.2 mm, vias 0 -> 4
- net GND: track 0.52 -> 121.6 mm, vias 157 -> 43
- net /EMS/Relay_Signal_OUT: track 0.00 -> 95.3 mm, vias 0 -> 6
- net /PWR_Cutoff_Relay Sheet/Relay_Coil_Signal: track 90.0 -> 0.00 mm, vias 4 -> 0
- net +12V: track 64.2 -> 137.2 mm, vias 0 -> 2
- net +5V: track 0.00 -> 60.8 mm, vias 0 -> 6
- net MCU_running: track 0.00 -> 49.9 mm, vias 0 -> 8
- net Net-(SW4-B): track 0.00 -> 45.0 mm, vias 0 -> 2
- net Net-(J1-Pin_3): track 0.00 -> 35.7 mm
- net Net-(J1-Pin_4): track 0.00 -> 34.2 mm
- net /EMS/MCU_EMS_Observe: track 0.00 -> 30.9 mm, vias 0 -> 4
- net /EMS/MCU_EMC_signal: track 0.00 -> 28.0 mm, vias 0 -> 4
- net Net-(SW3-B): track 0.00 -> 27.5 mm
- net /STM32F103/CAN_ID4: track 0.00 -> 26.5 mm, vias 0 -> 2
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- added copper zone on F.Cu, net +5V
- added copper zone on F.Cu, net Actuator_Power
- added copper zone on F.Cu, net Logic_line_Power
- added copper zone on F.Cu, net Net-(D8-K)
- removed copper zone on B.Cu, net GNDPWR
- removed copper zone on F.Cu, net GNDPWR
Other:
- board text added: "CAN ID"
- board text added: "Power Supply Board v0.2"
- board text added: "Powers"
- board text added: "RESET"
- board text added: "Relays"
- board text added: "STM32 Operation"
- board text added: "STlink"
- board text removed: "12V IN"
- board text removed: "Bat"
- board text removed: "Logic indicators"
- board text removed: "MCU Board"
- board text removed: "Power Supply Board v0.1"
- board text removed: "Power indicator"
- board text removed: "Voltage measurement"
- board text removed: "Warning! Disconnect at 24V!"
- board text removed: "Warning! Disconnect when attaching MCU board!"
